File: projects/TEST_KICAD1/TEST_KICAD1.kicad_pcb (KiCad board)
At the start: 2 copper layers, 37 x 41 mm, 17 parts, among them J3 FTDI, SW1 SW_Push, U1 ATmega328P-A, Y1 16MHz

Commit message: fin PCb, bom
Parts:
- added G***: LOGO, MyLibraryFootprint:MLF_Croco, F.Cu at (81.0, 100.5)
- C1, C2: value 12pF -> C
- C3, C4, C5: value 100nF -> C
- C6: value 1uF -> C
- D1: value Green -> LED
- D2: value Red -> LED
- R1: value 33Ω -> R
- R2, R3: value 10K -> R
- Y1: value 16MHz -> Crystal
