File: projects/TEST_KICAD1/TEST_KICAD1.kicad_sch (KiCad schematic)
At the start: 17 parts, among them J3 FTDI, SW1 SW_Push, U1 ATmega328P-A, Y1 16MHz

Commit message: link footprint-symbol
Parts:
- C1, C2, C3, C4, C5, C6, R1, R2, R3: footprint (none) -> MyLibraryFootprint:MLF-CapacitorResistor-0603-1608mm
- D1, D2: footprint (none) -> MyLibraryFootprint:MLF-LED-0603-1608mm
- J1: footprint (none) -> MyLibraryFootprint:MLF-J
- J2: footprint (none) -> MyLibraryFootprint:MLF-J2
- J3: footprint (none) -> MyLibraryFootprint:MLF-J3
- SW1: footprint (none) -> MyLibraryFootprint:MLF-Switch_button_B3U-1000P
- U1: footprint (none) -> MyLibraryFootprint:MLF-ATmega328P-AU-32Av3
- Y1: footprint (none) -> MyLibraryFootprint:MLF-Crystal
Changed lines of the file:
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@@
 			)
 		)
-		(property "Footprint" ""
+		(property "Footprint" "MyLibraryFootprint:MLF-J"
 			(at 190.5 111.76 0)
 			(effects
@@
 	)
 	(symbol
+		(lib_name "C_3")
 		(lib_id "New_Library:C")
 		(at 153.67 114.3 90)
@@
 			)
 		)
-		(property "Footprint" ""
+		(property "Footprint" "MyLibraryFootprint:MLF-CapacitorResistor-0603-1608mm"
 			(at 153.67 114.3 0)
 			(effects
@@
 			)
 		)
-		(property "Footprint" ""
+		(property "Footprint" "MyLibraryFootprint:MLF-J3"
 			(at 240.03 113.03 0)
 			(effects
@@
 			)
 		)
-		(property "Footprint" ""
+		(property "Footprint" "MyLibraryFootprint:MLF-CapacitorResistor-0603-1608mm"
 			(at 240.03 35.56 0)
 			(effects
@@
 	)
 	(symbol
+		(lib_name "C_2")
 		(lib_id "New_Library:C")
 		(at 76.2 44.45 180)
@@
 			)
 		)
-		(property "Footprint" ""
+		(property "Footprint" "MyLibraryFootprint:MLF-CapacitorResistor-0603-1608mm"
 			(at 76.2 44.45 0)
 			(effects
@@
 			)
 		)
-		(property "Footprint" ""
+		(property "Footprint" "MyLibraryFootprint:MLF-Crystal"
 			(at 143.51 125.73 0)
 			(effects
@@
 			)
 		)
-		(property "Footprint" ""
+		(property "Footprint" "MyLibraryFootprint:MLF-LED-0603-1608mm"
 			(at 95.25 39.37 0)
 			(effects
@@
 	)
 	(symbol
+		(lib_name "C_5")
 		(lib_id "New_Library:C")
 		(at 34.29 133.35 90)
@@
 			)
 		)
-		(property "Footprint" ""
+		(property "Footprint" "MyLibraryFootprint:MLF-CapacitorResistor-0603-1608mm"
 			(at 34.29 133.35 0)
 			(effects
@@
 			)
 		)
-		(property "Footprint" ""
+		(property "Footprint" "MyLibraryFootprint:MLF-Switch_button_B3U-1000P"
 			(at 227.33 43.18 0)
 			(effects
@@
 	)
 	(symbol
+		(lib_name "R_2")
 		(lib_id "New_Library:R")
 		(at 95.25 52.07 0)
@@
 			)
 		)
-		(property "Footprint" ""
+		(property "Footprint" "MyLibraryFootprint:MLF-CapacitorResistor-0603-1608mm"
 			(at 95.25 52.07 0)
 			(effects
@@
 	)
 	(symbol
+		(lib_name "C_4")
 		(lib_id "New_Library:C")
 		(at 153.67 139.7 90)
@@
 			)
 		)
-		(property "Footprint" ""
+		(property "Footprint" "MyLibraryFootprint:MLF-CapacitorResistor-0603-1608mm"
 			(at 153.67 139.7 0)
 			(effects
@@
 	)
 	(symbol
+		(lib_name "LED_1")
 		(lib_id "New_Library:LED")
 		(at 148.59 48.26 90)
@@
 			)
 		)
-		(property "Footprint" ""
+		(property "Footprint" "MyLibraryFootprint:MLF-LED-0603-1608mm"
 			(at 148.59 48.26 0)
 			(effects
@@
 			)
 		)
-		(property "Footprint" ""
+		(property "Footprint" "MyLibraryFootprint:MLF-ATmega328P-AU-32Av3"
 			(at 76.2 134.62 0)
 			(effects
@@
 	)
 	(symbol
+		(lib_name "R_1")
 		(lib_id "New_Library:R")
 		(at 148.59 34.29 0)
@@
 			)
 		)
-		(property "Footprint" ""
+		(property "Footprint" "MyLibraryFootprint:MLF-CapacitorResistor-0603-1608mm"
 			(at 148.59 34.29 0)
 			(effects
@@
 			)
 		)
-		(property "Footprint" ""
+		(property "Footprint" "MyLibraryFootprint:MLF-J2"
 			(at 218.44 111.76 0)
 			(effects
@@
 			)
 		)
-		(property "Footprint" ""
+		(property "Footprint" "MyLibraryFootprint:MLF-CapacitorResistor-0603-1608mm"
 			(at 210.82 43.18 0)
 			(effects
@@
 	)
 	(symbol
+		(lib_name "C_1")
 		(lib_id "New_Library:C")
 		(at 58.42 44.45 0)
@@
 			)
 		)
-		(property "Footprint" ""
+		(property "Footprint" "MyLibraryFootprint:MLF-CapacitorResistor-0603-1608mm"
 			(at 58.42 44.45 0)
 			(effects

Commit message: ajout PCB
Connections:
- net GND: now also D1.1 (K); no longer D1.2 (A)
- net VCC: now also D2.2 (A); no longer D2.1 (K)
- net at R2.1: now also D2.1 (K); no longer D2.2 (A)
- net at R1.2: now also D1.2 (A); no longer D1.1 (K)
Changed lines of the file:
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@@
 	)
 	(symbol
-		(lib_name "J_1")
 		(lib_id "New_Library:J")
 		(at 190.5 111.76 180)
@@
 	)
 	(symbol
-		(lib_name "C_3")
 		(lib_id "New_Library:C")
 		(at 153.67 114.3 90)
@@
 	)
 	(symbol
-		(lib_name "C_2")
 		(lib_id "New_Library:C")
 		(at 76.2 44.45 180)
@@
 	)
 	(symbol
-		(lib_name "C_5")
 		(lib_id "New_Library:C")
 		(at 34.29 133.35 90)
@@
 	)
 	(symbol
-		(lib_name "R_2")
 		(lib_id "New_Library:R")
 		(at 95.25 52.07 0)
@@
 	)
 	(symbol
-		(lib_name "C_4")
 		(lib_id "New_Library:C")
 		(at 153.67 139.7 90)
@@
 	)
 	(symbol
-		(lib_name "LED_1")
 		(lib_id "New_Library:LED")
 		(at 148.59 48.26 90)
@@
 	)
 	(symbol
-		(lib_name "R_1")
 		(lib_id "New_Library:R")
 		(at 148.59 34.29 0)
@@
 	)
 	(symbol
-		(lib_name "C_1")
 		(lib_id "New_Library:C")
 		(at 58.42 44.45 0)

Commit message: fin PCb, bom
Parts:
- C1, C2: value 12pF -> C
- C3, C4, C5: value 100nF -> C
- C6: value 1uF -> C
- D1: value Green -> LED
- D2: value Red -> LED
- R1: value 33Ω -> R
- R2, R3: value 10K -> R
- SW1: Caracteristiques (none) -> 12V 2.5mm Round Button 3mm SPST 50mA SMD,3x2.5mm Tactile Sw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; Manufacture Part Number (none) -> B3U-1000P
- Y1: value 16MHz -> Crystal
Other:
- company: (none) ->  42Chips - Ecole 42
- title: (none) -> cgranja-piscineElec-design
